Commit message: added apartment scanning functionality

File: config/tiago_webots_mapping.urdf (robot description, URDF)
Before this commit: robot Tiago Webots, 1 links, 0 joints
Links:
- added link wheel_left_link
- added link wheel_right_link
Joints:
- added joint wheel_left_joint: type continuous, parent base_link, child wheel_left_link, origin xyz=0 0.2022 0, axis 0 1 0
- added joint wheel_right_joint: type continuous, parent base_link, child wheel_right_link, origin xyz=0 -0.2022 0, axis 0 1 0
